File: schematic/esp8266-01 carrier.brd (EAGLE design)
At the start: 69.5 x 22.8 mm, 17 parts, among them U1 WIRELESS-WIFI-ESP-01

Commit message: Added USB, gitignore
Parts:
- added CN1: (no value), adafruit:USB-MINIB-THM
Connections:
- net GND: now also CN1.GND
- net N$3: now also CN1.VBUS
Routing:
- net N$3: track 45.8 -> 67.4 mm
- net 3V3: track 86.0 -> 72.2 mm
- net GND: track 103.3 -> 117.1 mm
- net N$5: track 40.0 -> 33.5 mm
- net N$2: track 55.4 -> 49.0 mm
- net TX-GPIO1: track 32.4 -> 30.3 mm
- net N$1: track 10.2 -> 8.69 mm
- net N$6: track 45.8 -> 47.3 mm
- net N$4: track 34.6 -> 33.9 mm
Other:
- board size 69.5 x 22.8 mm -> 78.4 x 22.8 mm
- board text added: "Install R1, R2 with 5V UART"
- board text added: "UART"
