File: schematic/esp8266-01 carrier.sch (EAGLE design)
At the start: 17 parts, among them U1 WIRELESS-WIFI-ESP-01

Commit message: Added USB, gitignore
Parts:
- added CN1: (no value), adafruit:USBTHM
Connections:
- net GND: now also CN1.GND
- net N$3: now also CN1.VBUS
Changed lines of the file:
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@@
 <part name="JP4" library="adafruit" deviceset="PINHD-1X1" device=""/>
 <part name="JP5" library="adafruit" deviceset="PINHD-1X1" device=""/>
+<part name="CN1" library="adafruit" library_urn="urn:adsk.eagle:library:420" deviceset="USB" device="THM" package3d_urn="urn:adsk.eagle:package:6240695/1"/>
 </parts>
 <sheets>
@@
 <attribute name="VALUE" x="107.95" y="38.1" size="1.778" layer="96"/>
 </instance>
+<instance part="CN1" gate="G$1" x="60.96" y="43.18" smashed="yes">
+<attribute name="NAME" x="50.8" y="51.816" size="1.27" layer="95"/>
+<attribute name="VALUE" x="50.8" y="33.02" size="1.27" layer="96"/>
+</instance>
 </instances>
 <busses>
@@
 <junction x="152.4" y="43.18"/>
 <pinref part="JP1" gate="A" pin="2"/>
-<wire x1="93.98" y1="60.96" x2="62.992" y2="60.96" width="0.1524" layer="91"/>
+<wire x1="93.98" y1="60.96" x2="78.74" y2="60.96" width="0.1524" layer="91"/>
 <junction x="93.98" y="60.96"/>
 <pinref part="U1" gate="G$1" pin="GND"/>
 <pinref part="MGT3" gate="G$1" pin="P$1"/>
+<wire x1="78.74" y1="60.96" x2="62.992" y2="60.96" width="0.1524" layer="91"/>
 <wire x1="180.34" y1="43.18" x2="190.5" y2="43.18" width="0.1524" layer="91"/>
 <junction x="180.34" y="43.18"/>
@@
 <pinref part="JP5" gate="G$1" pin="1"/>
 <wire x1="111.76" y1="43.18" x2="124.46" y2="43.18" width="0.1524" layer="91"/>
+<pinref part="CN1" gate="G$1" pin="GND"/>
+<wire x1="71.12" y1="38.1" x2="78.74" y2="38.1" width="0.1524" layer="91"/>
+<wire x1="78.74" y1="38.1" x2="78.74" y2="60.96" width="0.1524" layer="91"/>
+<junction x="78.74" y="60.96"/>
 </segment>
 </net>
@@
 <pinref part="JP3" gate="A" pin="3"/>
 <pinref part="JP1" gate="A" pin="3"/>
-<wire x1="93.98" y1="58.42" x2="62.992" y2="58.42" width="0.1524" layer="91"/>
-</segment>
-</net>
+<wire x1="93.98" y1="58.42" x2="73.66" y2="58.42" width="0.1524" layer="91"/>
+<pinref part="CN1" gate="G$1" pin="VBUS"/>
+<wire x1="73.66" y1="58.42" x2="62.992" y2="58.42" width="0.1524" layer="91"/>
+<wire x1="71.12" y1="48.26" x2="73.66" y2="48.26" width="0.1524" layer="91"/>
+<wire x1="73.66" y1="48.26" x2="73.66" y2="58.42" width="0.1524" layer="91"/>
+<junction x="73.66" y="58.42"/>
+</segment>
+</net>
